Commit message: camera update
visual

File: sim/sim_vision/urdf/camera.xacro (robot description, xacro)
@@ -1,25 +1,47 @@
 <?xml version="1.0"?>
 <robot name="simple_camera" xmlns:xacro="http://www.ros.org/wiki/xacro">
-    <!-- Camera link (physical body) -->
-    <link name="camera_link">
-        <visual>
-            <geometry>
-                <box size="0.05 0.05 0.05"/>
-            </geometry>
-            <material name="black">
-                <color rgba="0 0 0 1"/>
-            </material>
-        </visual>
-        <collision>
-            <geometry>
-                <box size="0.05 0.05 0.05"/>
-            </geometry>
-        </collision>
-        <inertial>
-            <mass value="0.1"/>
-            <inertia ixx="0.0001" ixy="0" ixz="0"
-                    iyy="0.0001" iyz="0"
-                    izz="0.0001"/>
-        </inertial>
-    </link>
+  <xacro:include filename="$(find sim_vision)/urdf/materials.xacro" />
+  <link name="world"/>
+  <joint type="fixed" name="camera_joint">
+    <origin xyz="-0.6 0 1.63" rpy="0 0.86 0"/>
+    <child link="camera_link"/>
+    <parent link="world"/>
+  </joint>
+  <link name='camera_link'>
+    <pose>0 0 0 0 0 0</pose>
+    <inertial>
+      <mass value="1.0e-03"/>
+      <origin xyz="0 0 0" rpy="0 0 0"/>
+      <inertia
+          ixx="1e-6" ixy="0" ixz="0"
+          iyy="1e-6" iyz="0"
+          izz="1e-6"
+      />
+    </inertial>
+    <visual name="camera_body_visual">
+      <origin xyz="0 0 0" rpy="0 0 0"/>
+      <geometry>
+        <box size=".1 .05 .05"/>
+      </geometry>
+      <material name = "red">
+        <color rgba="0.8 0.0 0.0 1.0"/>
+      </material>
+    </visual>
+    <visual name="camera_lens_visual">
+      <origin xyz="0.06 0 0" rpy="0 0 0"/>
+      <geometry>
+        <sphere radius="0.015"/>
+      </geometry>
+      <material name = "blue">
+        <color rgba="0 0.0 0.8 1.0"/>
+      </material>
+    </visual>
+  </link>
+  <joint type="fixed" name="camera_optical_joint">
+    <origin xyz="0 0 0" rpy="-1.5707 0 -1.5707"/>
+    <child link="camera_link_optical"/>
+    <parent link="camera_link"/>
+  </joint>
+  <link name="camera_link_optical">
+  </link>
 </robot>

Commit message: spawn camera from xacro file

File: sim/sim_vision/urdf/camera.xacro (robot description, xacro)
@@ -1,5 +1,4 @@
 <?xml version="1.0"?>
 <robot name="simple_camera" xmlns:xacro="http://www.ros.org/wiki/xacro">
-  <xacro:include filename="$(find sim_vision)/urdf/materials.xacro" />
   <link name="world"/>
   <joint type="fixed" name="camera_joint">
@@ -38,10 +37,20 @@
     </visual>
   </link>
-  <joint type="fixed" name="camera_optical_joint">
-    <origin xyz="0 0 0" rpy="-1.5707 0 -1.5707"/>
-    <child link="camera_link_optical"/>
-    <parent link="camera_link"/>
-  </joint>
-  <link name="camera_link_optical">
-  </link>
+  <gazebo reference="camera_link">
+    <sensor name="camera" type="camera">
+      <camera>
+        <horizontal_fov>1.047</horizontal_fov>
+        <image>
+          <width>1280</width>
+          <height>720</height>
+          <format>R8G8B8</format>
+        </image>
+        <camera_info_topic>camera/camera_info</camera_info_topic>
+      </camera>
+      <always_on>true</always_on>
+      <update_rate>30</update_rate>
+      <visualize>true</visualize>
+      <topic>camera/image</topic>
+    </sensor>
+  </gazebo>
 </robot>
