Commit message: added camera_link to workspace.xacro

File: workspace_sim/urdf/workspace.xacro (robot description, xacro)
@@ -1,4 +1,4 @@
 <?xml version="1.0"?>
-<robot name="simple_camera" xmlns:xacro="http://www.ros.org/wiki/xacro">
+<robot name="workspace" xmlns:xacro="http://www.ros.org/wiki/xacro">
   <link name="world"/>
   <joint type="fixed" name="workspace_joint">
@@ -7,4 +7,30 @@
     <parent link="world"/>
   </joint>
-  <link name='workspace_link'/>
+  <link name='workspace_link'>
+    <inertial>
+      <mass value="1.0e-03"/>
+      <origin xyz="0 0 0" rpy="0 0 0"/>
+      <inertia
+          ixx="1e-6" ixy="0" ixz="0"
+          iyy="1e-6" iyz="0"
+          izz="1e-6"
+      />
+    </inertial>
+  </link>
+  <joint type="fixed" name="camera_joint">
+    <origin xyz="0 0 1" rpy="0 0 0"/>
+    <child link="camera_link"/>
+    <parent link="workspace_link"/>
+  </joint>
+  <link name='camera_link'>
+    <inertial>
+      <mass value="1.0e-03"/>
+      <origin xyz="-0.6 0 1.63" rpy="0 0.86 0"/>
+      <inertia
+          ixx="1e-6" ixy="0" ixz="0"
+          iyy="1e-6" iyz="0"
+          izz="1e-6"
+      />
+    </inertial>
+  </link>
 </robot>

Commit message: added ur5e to workspace.xacro

File: workspace_sim/urdf/workspace.xacro (robot description, xacro)
@@ -1,4 +1,10 @@
 <?xml version="1.0"?>
 <robot name="workspace" xmlns:xacro="http://www.ros.org/wiki/xacro">
+  <xacro:include filename="$(find ur_description)/urdf/ur_macro.xacro"/>
+  <xacro:arg name="ur_type" default="ur5e"/>
+  <xacro:arg name="joint_limits_parameters_file" default="$(find ur_description)/config/$(arg ur_type)/joint_limits.yaml"/>
+  <xacro:arg name="kinematics_parameters_file" default="$(find ur_description)/config/$(arg ur_type)/default_kinematics.yaml"/>
+  <xacro:arg name="physical_parameters_file" default="$(find ur_description)/config/$(arg ur_type)/physical_parameters.yaml"/>
+  <xacro:arg name="visual_parameters_file" default="$(find ur_description)/config/$(arg ur_type)/visual_parameters.yaml"/>
   <link name="world"/>
   <joint type="fixed" name="workspace_joint">
@@ -34,3 +40,20 @@
     </inertial>
   </link>
+  <link name="robot_mount"/>
+  <joint name="base_to_robot_mount" type="fixed">
+    <parent link="workspace_link"/>
+    <child link="robot_mount"/>
+    <origin xyz="0.845 0.85 0" rpy="0 0 ${pi}" />
+  </joint>
+  <xacro:ur_robot
+    name="$(arg ur_type)"
+    tf_prefix="$(arg ur_type)_"
+    parent="robot_mount"
+    joint_limits_parameters_file="$(arg joint_limits_parameters_file)"
+    kinematics_parameters_file="$(arg kinematics_parameters_file)"
+    physical_parameters_file="$(arg physical_parameters_file)"
+    visual_parameters_file="$(arg visual_parameters_file)"
+  >
+      <origin xyz="0 0 0" rpy="0 0 0" />
+  </xacro:ur_robot>
 </robot>
