Commit message: working ur5e spawn

File: workspace_sim/urdf/workspace.urdf.xacro (robot description, xacro)
@@ -1,10 +1,20 @@
 <?xml version="1.0"?>
-<robot name="workspace" xmlns:xacro="http://www.ros.org/wiki/xacro">
+<robot name="$(arg name)" xmlns:xacro="http://www.ros.org/wiki/xacro">
+  <xacro:arg name="name" default="ur"/>
   <xacro:include filename="$(find ur_description)/urdf/ur_macro.xacro"/>
-  <xacro:arg name="ur_type" default="ur5e"/>
-  <xacro:arg name="joint_limits_parameters_file" default="$(find ur_description)/config/$(arg ur_type)/joint_limits.yaml"/>
-  <xacro:arg name="kinematics_parameters_file" default="$(find ur_description)/config/$(arg ur_type)/default_kinematics.yaml"/>
-  <xacro:arg name="physical_parameters_file" default="$(find ur_description)/config/$(arg ur_type)/physical_parameters.yaml"/>
-  <xacro:arg name="visual_parameters_file" default="$(find ur_description)/config/$(arg ur_type)/visual_parameters.yaml"/>
+  <xacro:include filename="$(find ur_simulation_gz)/urdf/ur_gz.ros2_control.xacro" />
+  <xacro:arg name="ur_type" default="ur5x"/>
+  <!-- parameters -->
+  <xacro:arg name="tf_prefix" default="" />
+  <xacro:arg name="joint_limit_params" default="$(find ur_description)/config/$(arg ur_type)/joint_limits.yaml"/>
+  <xacro:arg name="kinematics_params" default="$(find ur_description)/config/$(arg ur_type)/default_kinematics.yaml"/>
+  <xacro:arg name="physical_params" default="$(find ur_description)/config/$(arg ur_type)/physical_parameters.yaml"/>
+  <xacro:arg name="visual_params" default="$(find ur_description)/config/$(arg ur_type)/visual_parameters.yaml"/>
+  <xacro:arg name="transmission_hw_interface" default=""/>
+  <xacro:arg name="safety_limits" default="false"/>
+  <xacro:arg name="safety_pos_margin" default="0.15"/>
+  <xacro:arg name="safety_k_position" default="20"/>
+  <xacro:arg name="simulation_controllers" default="" />
+  <xacro:arg name="ros_namespace" default="" />
   <link name="world"/>
   <joint type="fixed" name="workspace_joint">
@@ -44,16 +54,37 @@
     <parent link="workspace_link"/>
     <child link="robot_mount"/>
-    <origin xyz="0.845 0.85 0" rpy="0 0 ${pi}" />
+    <origin xyz="0.5 0 0" rpy="0 0 ${pi}" />
   </joint>
+  <!-- arm -->
   <xacro:ur_robot
-    name="$(arg ur_type)"
-    tf_prefix="$(arg ur_type)_"
+    name="$(arg name)"
+    tf_prefix="$(arg tf_prefix)"
     parent="robot_mount"
-    joint_limits_parameters_file="$(arg joint_limits_parameters_file)"
-    kinematics_parameters_file="$(arg kinematics_parameters_file)"
-    physical_parameters_file="$(arg physical_parameters_file)"
-    visual_parameters_file="$(arg visual_parameters_file)"
-  >
-      <origin xyz="0 0 0" rpy="0 0 0" />
+    joint_limits_parameters_file="$(arg joint_limit_params)"
+    kinematics_parameters_file="$(arg kinematics_params)"
+    physical_parameters_file="$(arg physical_params)"
+    visual_parameters_file="$(arg visual_params)"
+    safety_limits="$(arg safety_limits)"
+    safety_pos_margin="$(arg safety_pos_margin)"
+    safety_k_position="$(arg safety_k_position)"
+    force_abs_paths="true"
+    >
+    <origin xyz="0 0 0" rpy="0 0 0" />          <!-- position robot in the world -->
   </xacro:ur_robot>
+  <gazebo reference="world">
+  </gazebo>
+  <gazebo>
+    <plugin filename="gz_ros2_control-system" name="gz_ros2_control::GazeboSimROS2ControlPlugin">
+      <parameters>$(arg simulation_controllers)</parameters>
+      <ros>
+        <namespace>$(arg ros_namespace)</namespace>
+      </ros>
+    </plugin>
+  </gazebo>
+  <!-- ros2 control instance -->
+  <xacro:ur_ros2_control
+    name="$(arg name)"
+    tf_prefix="$(arg tf_prefix)"
+    transmission_hw_interface="$(arg transmission_hw_interface)"
+  />
 </robot>

Commit message: adjusted workspace_link

File: workspace_sim/urdf/workspace.urdf.xacro (robot description, xacro)
@@ -19,5 +19,5 @@
   <link name="world"/>
   <joint type="fixed" name="workspace_joint">
-    <origin xyz="0 0 1" rpy="0 0 0"/>
+    <origin xyz="0 0 1" rpy="0 0 -1.5708"/>
     <child link="workspace_link"/>
     <parent link="world"/>
@@ -54,5 +54,5 @@
     <parent link="workspace_link"/>
     <child link="robot_mount"/>
-    <origin xyz="0.5 0 0" rpy="0 0 ${pi}" />
+    <origin xyz="0 0.5 0" rpy="0 0 ${pi}" />
   </joint>
   <!-- arm -->
