Commit message: updated robot_arm_moveit.urdf.xacro

File: workspace_sim/urdf/robot_arm_moveit.urdf.xacro (robot description, xacro)
@@ -2,5 +2,7 @@
 <robot name="ur" xmlns:xacro="http://www.ros.org/wiki/xacro">
   <xacro:include filename="$(find ur_description)/urdf/ur_macro.xacro"/>
-  <xacro:include filename="$(find ur_simulation_gz)/urdf/ur_gz.ros2_control.xacro" />
+  <xacro:include filename="$(find rh_p12_rn_description)/urdf/rh_p12_rn_macro.xacro"/>
+  <xacro:include filename="$(find ur_description)/urdf/inc/ur_joint_control.xacro" />
+  <xacro:include filename="$(find rh_p12_rn_description)/urdf/joint_control.xacro" />
   <xacro:arg name="ur_type" default="ur5e"/>
   <!-- parameters -->
@@ -71,3 +73,29 @@
     <origin xyz="0 0 0" rpy="0 0 0" />          <!-- position robot in the world -->
   </xacro:ur_robot>
+  <xacro:rh_p12_rn parent="$(arg tf_prefix)tool0"/>
+  <!-- End effector -->
+  <joint name="end_effector_joint" type="fixed">
+    <origin xyz="0.0 0.0 0.12" rpy="0 0 0"/>
+    <parent link="rh_p12_rn_base"/>
+    <child link="end_effector_link"/>
+  </joint>
+  <!-- End effector link -->
+  <link name="end_effector_link">
+    <visual>
+      <origin xyz="0 0 0" rpy="0 0 0"/>
+      <geometry>
+        <box size="0.01 0.01 0.01" />
+      </geometry>
+      <material name="red">
+        <color rgba="0.8 0.0 0.0 1.0"/>
+      </material>
+    </visual>
+    <inertial>
+      <origin xyz="0 0 0" />
+      <mass value="1.0e-03" />
+      <inertia ixx="1.0e-03" ixy="0.0" ixz="0.0"
+               iyy="1.0e-03" iyz="0.0"
+               izz="1.0e-03" />
+    </inertial>
+  </link>
 </robot>

Commit message: added back table collision to URDF

File: workspace_sim/urdf/robot_arm_moveit.urdf.xacro (robot description, xacro)
@@ -25,4 +25,10 @@
   </joint>
   <link name='workspace_link'>
+    <collision>
+      <origin xyz="0 0 -0.015" rpy="0 0 0"/>
+      <geometry>
+        <box size="0.8 1.5 0.03" />
+      </geometry>
+    </collision>
     <inertial>
       <mass value="1.0e-03"/>
