Commit message: moveit config

File: workspace_sim/urdf/robot_arm.urdf.xacro (robot description, xacro)
@@ -1,8 +1,7 @@
 <?xml version="1.0"?>
-<robot name="$(arg name)" xmlns:xacro="http://www.ros.org/wiki/xacro">
-  <xacro:arg name="name" default="ur"/>
+<robot name="ur" xmlns:xacro="http://www.ros.org/wiki/xacro">
   <xacro:include filename="$(find ur_description)/urdf/ur_macro.xacro"/>
   <xacro:include filename="$(find ur_simulation_gz)/urdf/ur_gz.ros2_control.xacro" />
-  <xacro:arg name="ur_type" default="ur5x"/>
+  <xacro:arg name="ur_type" default="ur5e"/>
   <!-- parameters -->
   <xacro:arg name="tf_prefix" default="" />
@@ -58,5 +57,5 @@
   <!-- arm -->
   <xacro:ur_robot
-    name="$(arg name)"
+    name="ur"
     tf_prefix="$(arg tf_prefix)"
     parent="robot_mount"

File: workspace_sim/urdf/robot_arm_moveit.urdf.xacro (robot description, xacro)
@@ -1,5 +1,6 @@
 <?xml version="1.0"?>
 <robot name="ur" xmlns:xacro="http://www.ros.org/wiki/xacro">
-  <xacro:include filename="$(find workspace_sim)/urdf/robot_arm_moveit_macro.xacro"/>
+  <xacro:include filename="$(find ur_description)/urdf/ur_macro.xacro"/>
+  <xacro:include filename="$(find ur_simulation_gz)/urdf/ur_gz.ros2_control.xacro" />
   <xacro:arg name="ur_type" default="ur5e"/>
   <!-- parameters -->
@@ -13,8 +14,50 @@
   <xacro:arg name="safety_pos_margin" default="0.15"/>
   <xacro:arg name="safety_k_position" default="20"/>
+  <xacro:arg name="simulation_controllers" default="" />
+  <xacro:arg name="ros_namespace" default="" />
   <link name="world"/>
-  <xacro:robot_arm
-    parent="world"
-    ur_type="$(arg ur_type)"
+  <joint type="fixed" name="workspace_joint">
+    <origin xyz="0 0 1" rpy="0 0 -1.5708"/>
+    <child link="workspace_link"/>
+    <parent link="world"/>
+  </joint>
+  <link name='workspace_link'>
+    <inertial>
+      <mass value="1.0e-03"/>
+      <origin xyz="0 0 0" rpy="0 0 0"/>
+      <inertia
+          ixx="1e-6" ixy="0" ixz="0"
+          iyy="1e-6" iyz="0"
+          izz="1e-6"
+      />
+    </inertial>
+  </link>
+  <joint type="fixed" name="camera_joint">
+    <origin xyz="0 0 1" rpy="0 0 0"/>
+    <child link="camera_link"/>
+    <parent link="workspace_link"/>
+  </joint>
+  <link name='camera_link'>
+    <inertial>
+      <mass value="1.0e-03"/>
+      <origin xyz="-0.6 0 1.63" rpy="0 0.86 0"/>
+      <inertia
+          ixx="1e-6" ixy="0" ixz="0"
+          iyy="1e-6" iyz="0"
+          izz="1e-6"
+      />
+    </inertial>
+  </link>
+  <link name="robot_mount"/>
+  <joint name="base_to_robot_mount" type="fixed">
+    <parent link="workspace_link"/>
+    <child link="robot_mount"/>
+    <origin xyz="0 0.5 0" rpy="0 0 ${pi}" />
+  </joint>
+  <!-- arm -->
+  <xacro:ur_robot
+    name="ur"
+    tf_prefix="$(arg tf_prefix)"
+    parent="robot_mount"
     joint_limits_parameters_file="$(arg joint_limit_params)"
     kinematics_parameters_file="$(arg kinematics_params)"
@@ -24,6 +67,7 @@
     safety_pos_margin="$(arg safety_pos_margin)"
     safety_k_position="$(arg safety_k_position)"
+    force_abs_paths="true"
     >
-      <origin xyz="0 0 1" rpy="0 0 -1.5708"/>
-  </xacro:robot_arm>
+    <origin xyz="0 0 0" rpy="0 0 0" />          <!-- position robot in the world -->
+  </xacro:ur_robot>
 </robot>

Commit message: end effector

File: workspace_sim/urdf/robot_arm.urdf.xacro (robot description, xacro)
@@ -74,4 +74,29 @@
   </xacro:ur_robot>
   <xacro:rh_p12_rn parent="$(arg tf_prefix)tool0"/>
+  <!-- End effector -->
+  <joint name="end_effector_joint" type="fixed">
+    <origin xyz="0.0 0.0 0.12" rpy="0 0 0"/>
+    <parent link="rh_p12_rn_base"/>
+    <child link="end_effector_link"/>
+  </joint>
+  <!-- End effector link -->
+  <link name="end_effector_link">
+    <visual>
+      <origin xyz="0 0 0" rpy="0 0 0"/>
+      <geometry>
+        <box size="0.01 0.01 0.01" />
+      </geometry>
+      <material name="red">
+        <color rgba="0.8 0.0 0.0 1.0"/>
+      </material>
+    </visual>
+    <inertial>
+      <origin xyz="0 0 0" />
+      <mass value="1.0e-03" />
+      <inertia ixx="1.0e-03" ixy="0.0" ixz="0.0"
+               iyy="1.0e-03" iyz="0.0"
+               izz="1.0e-03" />
+    </inertial>
+  </link>
   <gazebo reference="world">
   </gazebo>

Commit message: modified workspace_link in robot urdf
moved it to the table surface
added collision

File: workspace_sim/urdf/robot_arm.urdf.xacro (robot description, xacro)
@@ -20,9 +20,15 @@
   <link name="world"/>
   <joint type="fixed" name="workspace_joint">
-    <origin xyz="0 0 1" rpy="0 0 -1.5708"/>
+    <origin xyz="0 0 1.015" rpy="0 0 -1.5708"/>
     <child link="workspace_link"/>
     <parent link="world"/>
   </joint>
   <link name='workspace_link'>
+    <collision>
+      <origin xyz="0 0 -0.015" rpy="0 0 0"/>
+      <geometry>
+        <box size="0.8 1.5 0.03" />
+      </geometry>
+    </collision>
     <inertial>
       <mass value="1.0e-03"/>

Commit message: removed workspace collision from robot urdf

File: workspace_sim/urdf/robot_arm.urdf.xacro (robot description, xacro)
@@ -25,10 +25,4 @@
   </joint>
   <link name='workspace_link'>
-    <collision>
-      <origin xyz="0 0 -0.015" rpy="0 0 0"/>
-      <geometry>
-        <box size="0.8 1.5 0.03" />
-      </geometry>
-    </collision>
     <inertial>
       <mass value="1.0e-03"/>

Commit message: regenerated moveit config
joint limits changed in urdf
removed ur_arm_gripper group
removed workspace collision

File: workspace_sim/urdf/robot_arm.urdf.xacro (robot description, xacro)
@@ -8,5 +8,5 @@
   <!-- parameters -->
   <xacro:arg name="tf_prefix" default="" />
-  <xacro:arg name="joint_limit_params" default="$(find ur_description)/config/$(arg ur_type)/joint_limits.yaml"/>
+  <xacro:arg name="joint_limit_params" default="$(find workspace_sim)/config/joint_limits.yaml"/>
   <xacro:arg name="kinematics_params" default="$(find ur_description)/config/$(arg ur_type)/default_kinematics.yaml"/>
   <xacro:arg name="physical_params" default="$(find ur_description)/config/$(arg ur_type)/physical_parameters.yaml"/>

File: workspace_sim/urdf/robot_arm_moveit.urdf.xacro (robot description, xacro)
@@ -8,5 +8,5 @@
   <!-- parameters -->
   <xacro:arg name="tf_prefix" default="" />
-  <xacro:arg name="joint_limit_params" default="$(find ur_description)/config/$(arg ur_type)/joint_limits.yaml"/>
+  <xacro:arg name="joint_limit_params" default="$(find workspace_sim)/config/joint_limits.yaml"/>
   <xacro:arg name="kinematics_params" default="$(find ur_description)/config/$(arg ur_type)/default_kinematics.yaml"/>
   <xacro:arg name="physical_params" default="$(find ur_description)/config/$(arg ur_type)/physical_parameters.yaml"/>
@@ -25,10 +25,4 @@
   </joint>
   <link name='workspace_link'>
-    <collision>
-      <origin xyz="0 0 -0.015" rpy="0 0 0"/>
-      <geometry>
-        <box size="0.8 1.5 0.03" />
-      </geometry>
-    </collision>
     <inertial>
       <mass value="1.0e-03"/>

Commit message: move camera from world to robot model

File: workspace_sim/urdf/robot_arm.urdf.xacro (robot description, xacro)
@@ -99,4 +99,37 @@
     </inertial>
   </link>
+  <joint type="fixed" name="table_camera_joint">
+    <origin xyz="0 0 2.5" rpy="0 1.5707 0"/>
+    <child link="table_camera_link"/>
+    <parent link="world"/>
+  </joint>
+  <link name='table_camera_link'>
+    <pose>0 0 0 0 0 0</pose>
+    <inertial>
+      <mass value="1.0e-03"/>
+      <origin xyz="0 0 0" rpy="0 0 0"/>
+      <inertia
+          ixx="1e-6" ixy="0" ixz="0"
+          iyy="1e-6" iyz="0"
+          izz="1e-6"
+      />
+    </inertial>
+    <visual>
+      <origin xyz="0 0 0" rpy="0 0 0"/>
+      <geometry>
+        <box size=".05 .05 .05"/>
+      </geometry>
+      <material name="red">
+        <color rgba="0.0 0.0 0.8 1.0"/>
+      </material>
+    </visual>
+  </link>
+  <joint type="fixed" name="table_camera_optical_joint">
+    <origin xyz="0 0 0" rpy="-1.5707 0 -1.5707"/>
+    <child link="table_camera_link_optical"/>
+    <parent link="table_camera_link"/>
+  </joint>
+  <link name="table_camera_link_optical">
+  </link>
   <gazebo reference="world">
   </gazebo>
@@ -108,4 +141,34 @@
       </ros>
     </plugin>
+  </gazebo>
+  <gazebo reference="table_camera_link">
+    <sensor name="camera" type="camera">
+      <camera>
+        <horizontal_fov>1.047</horizontal_fov>
+        <image>
+          <width>1280</width>
+          <height>720</height>
+          <format>R8G8B8</format>
+        </image>
+        <clip>
+          <near>0.1</near>
+          <far>15</far>
+        </clip>
+        <noise>
+          <type>gaussian</type>
+          <!-- Noise is sampled independently per pixel on each frame.
+               That pixel's noise value is added to each of its color
+               channels, which at that point lie in the range [0,1]. -->
+          <mean>0.0</mean>
+          <stddev>0.007</stddev>
+        </noise>
+        <optical_frame_id>table_camera_link_optical</optical_frame_id>
+        <camera_info_topic>table_camera/camera_info</camera_info_topic>
+      </camera>
+      <always_on>1</always_on>
+      <update_rate>30</update_rate>
+      <visualize>true</visualize>
+      <topic>table_camera/image</topic>
+    </sensor>
   </gazebo>
   <!-- ros2 control instance -->

Commit message: modified robot model
camera position

File: workspace_sim/urdf/robot_arm.urdf.xacro (robot description, xacro)
@@ -100,5 +100,5 @@
   </link>
   <joint type="fixed" name="table_camera_joint">
-    <origin xyz="0 0 2.5" rpy="0 1.5707 0"/>
+    <origin xyz="-1.1 0 2.13" rpy="0 0.86 0"/>
     <child link="table_camera_link"/>
     <parent link="world"/>

Commit message: renamed camera_link to camera_link_optical

File: workspace_sim/urdf/robot_arm.urdf.xacro (robot description, xacro)
@@ -37,8 +37,8 @@
   <joint type="fixed" name="camera_joint">
     <origin xyz="0 0 1" rpy="0 0 0"/>
-    <child link="camera_link"/>
+    <child link="camera_link_optical"/>
     <parent link="workspace_link"/>
   </joint>
-  <link name='camera_link'>
+  <link name='camera_link_optical'>
     <inertial>
       <mass value="1.0e-03"/>
@@ -100,5 +100,5 @@
   </link>
   <joint type="fixed" name="table_camera_joint">
-    <origin xyz="-1.1 0 2.13" rpy="0 0.86 0"/>
+    <origin xyz="-1.1 -0.1 2.13" rpy="0 0.86 0"/>
     <child link="table_camera_link"/>
     <parent link="world"/>

Commit message: camera_extrinsic.py cleanup

File: workspace_sim/urdf/robot_arm.urdf.xacro (robot description, xacro)
@@ -35,5 +35,5 @@
     </inertial>
   </link>
-  <joint type="fixed" name="camera_joint">
+  <joint type="fixed" name="camera_joint_optical">
     <origin xyz="0 0 1" rpy="0 0 0"/>
     <child link="camera_link_optical"/>
@@ -43,5 +43,5 @@
     <inertial>
       <mass value="1.0e-03"/>
-      <origin xyz="-0.6 0 1.63" rpy="0 0.86 0"/>
+      <origin xyz="0 0 0" rpy="0 0 0"/>
       <inertia
           ixx="1e-6" ixy="0" ixz="0"

Commit message: rh_p12_rn_a custom decription package
urdf

File: workspace_sim/urdf/robot_arm.urdf.xacro (robot description, xacro)
@@ -5,4 +5,5 @@
   <xacro:include filename="$(find ur_description)/urdf/inc/ur_joint_control.xacro" />
   <xacro:include filename="$(find rh_p12_rn_description)/urdf/joint_control.xacro" />
+  <xacro:include filename="$(find rh_p12_rn_a_description_custom)/urdf/rh_p12_rn_a.xacro" />
   <xacro:arg name="ur_type" default="ur5e"/>
   <!-- parameters -->
@@ -73,5 +74,10 @@
     <origin xyz="0 0 0" rpy="0 0 0" />          <!-- position robot in the world -->
   </xacro:ur_robot>
-  <xacro:rh_p12_rn parent="$(arg tf_prefix)tool0"/>
+  <joint name="$(arg tf_prefix)gripper_joint" type="fixed">
+    <parent link="tool0"/>
+    <child link="$(arg tf_prefix)rh_p12_rn_base"/>
+    <origin xyz="0 0 0" rpy="0 0 0"/>
+  </joint>
+  <xacro:rh_p12_rn_a prefix="$(arg tf_prefix)" />
   <!-- End effector -->
   <joint name="end_effector_joint" type="fixed">
@@ -181,5 +187,4 @@
       initial_positions="${dict(shoulder_pan_joint=0.0,shoulder_lift_joint=-1.57,elbow_joint=0.0,wrist_1_joint=-1.57,wrist_2_joint=0.0,wrist_3_joint=0.0)}"
     />
-    <xacro:rh_p12_rn_joint_control_description/>
   </ros2_control>
 </robot>

Commit message: table camera parent is now workspac_link

File: workspace_sim/urdf/robot_arm.urdf.xacro (robot description, xacro)
@@ -110,7 +110,7 @@
   </link>
   <joint type="fixed" name="table_camera_joint">
-    <origin xyz="-1.1 -0.1 2.13" rpy="0 0.86 0"/>
+    <origin xyz="0.1 -1.1 1.115" rpy="0 0.86 1.5707"/>
     <child link="table_camera_link"/>
-    <parent link="world"/>
+    <parent link="workspace_link"/>
   </joint>
   <link name='table_camera_link'>
