Commit message: gripper update
added a joint
added gripper controller to config

File: rh_p12_rn_description/urdf/joint_control.xacro (robot description, xacro)
@@ -2,4 +2,15 @@
 <robot xmlns:xacro="http://wiki.ros.org/xacro">
   <xacro:macro name="rh_p12_rn_joint_control_description">
+	<joint name="rh_p12_rn">
+    <command_interface name="position">
+      <param name="min">-2</param>
+      <param name="max">2</param>
+    </command_interface>
+    <state_interface name="position">
+      <param name="initial_value">0.0</param>
+    </state_interface>
+    <state_interface name="velocity"/>
+    <state_interface name="effort"/>
+	</joint>
   </xacro:macro>
 </robot>

File: workspace_sim/urdf/robot_arm.urdf.xacro (robot description, xacro)
@@ -4,4 +4,5 @@
   <xacro:include filename="$(find rh_p12_rn_description)/urdf/rh_p12_rn_macro.xacro"/>
   <xacro:include filename="$(find ur_description)/urdf/inc/ur_joint_control.xacro" />
+  <xacro:include filename="$(find rh_p12_rn_description)/urdf/joint_control.xacro" />
   <xacro:arg name="ur_type" default="ur5e"/>
   <!-- parameters -->
@@ -92,4 +93,5 @@
       initial_positions="${dict(shoulder_pan_joint=0.0,shoulder_lift_joint=-1.57,elbow_joint=0.0,wrist_1_joint=-1.57,wrist_2_joint=0.0,wrist_3_joint=0.0)}"
     />
+    <xacro:rh_p12_rn_joint_control_description/>
   </ros2_control>
 </robot>

Commit message: gripper control

File: rh_p12_rn_description/urdf/joint_control.xacro (robot description, xacro)
@@ -13,4 +13,37 @@
     <state_interface name="effort"/>
 	</joint>
+	<joint name="rh_r2">
+    <command_interface name="position">
+      <param name="min">-2</param>
+      <param name="max">2</param>
+    </command_interface>
+    <state_interface name="position">
+      <param name="initial_value">0.0</param>
+    </state_interface>
+    <state_interface name="velocity"/>
+    <state_interface name="effort"/>
+	</joint>
+	<joint name="rh_l1">
+    <command_interface name="position">
+      <param name="min">-2</param>
+      <param name="max">2</param>
+    </command_interface>
+    <state_interface name="position">
+      <param name="initial_value">0.0</param>
+    </state_interface>
+    <state_interface name="velocity"/>
+    <state_interface name="effort"/>
+	</joint>
+	<joint name="rh_l2">
+    <command_interface name="position">
+      <param name="min">-2</param>
+      <param name="max">2</param>
+    </command_interface>
+    <state_interface name="position">
+      <param name="initial_value">0.0</param>
+    </state_interface>
+    <state_interface name="velocity"/>
+    <state_interface name="effort"/>
+	</joint>
   </xacro:macro>
 </robot>

File: rh_p12_rn_description/urdf/rh_p12_rn_macro.xacro (robot description, xacro)
@@ -39,14 +39,4 @@
             <dynamics damping="0.7"/>
         </joint>
-        <transmission name="tran_r1">
-            <type>transmission_interface/SimpleTransmission</type>
-            <joint name="rh_p12_rn">
-            <hardwareInterface>hardware_interface/EffortJointInterface</hardwareInterface>
-            </joint>
-            <actuator name="motor_r1">
-            <hardwareInterface>hardware_interface/EffortJointInterface</hardwareInterface>
-            <mechanicalReduction>1</mechanicalReduction>
-            </actuator>
-        </transmission>
         <!-- rh_p12_rn_r1 -->
         <link name="rh_p12_rn_r1">
@@ -80,14 +70,4 @@
             <dynamics damping="0.7"/>
         </joint>
-        <transmission name="tran_r2">
-            <type>transmission_interface/SimpleTransmission</type>
-            <joint name="rh_r2">
-            <hardwareInterface>hardware_interface/EffortJointInterface</hardwareInterface>
-            </joint>
-            <actuator name="motor_r2">
-            <hardwareInterface>hardware_interface/EffortJointInterface</hardwareInterface>
-            <mechanicalReduction>1</mechanicalReduction>
-            </actuator>
-        </transmission>
         <!-- rh_p12_rn_r2 -->
         <link name="rh_p12_rn_r2">
@@ -121,14 +101,4 @@
             <dynamics damping="0.7"/>
         </joint>
-        <transmission name="tran_l1">
-            <type>transmission_interface/SimpleTransmission</type>
-            <joint name="rh_l1">
-            <hardwareInterface>hardware_interface/EffortJointInterface</hardwareInterface>
-            </joint>
-            <actuator name="motor_l1">
-            <hardwareInterface>hardware_interface/EffortJointInterface</hardwareInterface>
-            <mechanicalReduction>1</mechanicalReduction>
-            </actuator>
-        </transmission>
         <!-- rh_p12_rn_l1 -->
         <link name="rh_p12_rn_l1">
@@ -162,14 +132,4 @@
             <dynamics damping="0.7"/>
         </joint>
-        <transmission name="tran_l2">
-            <type>transmission_interface/SimpleTransmission</type>
-            <joint name="rh_l2">
-            <hardwareInterface>hardware_interface/EffortJointInterface</hardwareInterface>
-            </joint>
-            <actuator name="motor_l2">
-            <hardwareInterface>hardware_interface/EffortJointInterface</hardwareInterface>
-            <mechanicalReduction>1</mechanicalReduction>
-            </actuator>
-        </transmission>
         <!-- rh_p12_rn_l2 -->
         <link name="rh_p12_rn_l2">
