Commit message: completed gripper model

File: rh_p12_rn_description/urdf/rh_p12_rn_macro.xacro (robot description, xacro)
@@ -31,11 +31,167 @@
         </link>
         <!-- Joint -->
-        <!--joint name="rh_p12_rn" type="revolute">
+        <joint name="rh_p12_rn" type="revolute">
             <parent link="rh_p12_rn_base"/>
+            <child link="rh_p12_rn_r1"/>
             <origin xyz="0.0 0.008 0.048" rpy="0 0 0"/>
             <axis xyz="1 0 0"/>
             <limit velocity="6.5" effort="1000" lower="0.0" upper="1.1" />
             <dynamics damping="0.7"/>
-        </joint-->
+        </joint>
+        <transmission name="tran_r1">
+            <type>transmission_interface/SimpleTransmission</type>
+            <joint name="rh_p12_rn">
+            <hardwareInterface>hardware_interface/EffortJointInterface</hardwareInterface>
+            </joint>
+            <actuator name="motor_r1">
+            <hardwareInterface>hardware_interface/EffortJointInterface</hardwareInterface>
+            <mechanicalReduction>1</mechanicalReduction>
+            </actuator>
+        </transmission>
+        <!-- rh_p12_rn_r1 -->
+        <link name="rh_p12_rn_r1">
+            <collision>
+            <origin xyz="0 0 0" rpy="0 0 0"/>
+            <geometry>
+                <mesh filename="file://$(find rh_p12_rn_description)/meshes/r1.stl" scale="0.001 0.001 0.001"/>
+            </geometry>
+            </collision>
+            <visual>
+            <origin xyz="0 0 0" rpy="0 0 0"/>
+            <geometry>
+                <mesh filename="file://$(find rh_p12_rn_description)/meshes/r1.stl" scale="0.001 0.001 0.001"/>
+            </geometry>
+            <material name="grey"/>
+            </visual>
+            <inertial>
+            <origin xyz="0.000 0.034 0.004" rpy="0 0 0"/>
+            <mass value="0.068"/>
+            <!--<inertia ixx="0.00004" ixy="0.0" ixz="0.0" iyy="0.00002" iyz="-0.00001" izz="0.00002" />-->
+            <inertia ixx="1.0" ixy="0.0" ixz="0.0" iyy="1.0" iyz="0.0" izz="1.0" />
+            </inertial>
+        </link>
+        <!-- Right Joint 2 -->
+        <joint name="rh_r2" type="revolute">
+            <parent link="rh_p12_rn_r1"/>
+            <child link="rh_p12_rn_r2"/>
+            <origin xyz="0.0 0.0493634 0.0285" rpy="0 0 0"/>
+            <axis xyz="-1 0 0"/>
+            <limit velocity="6.5" effort="1000" lower="0.0" upper="1.0" />
+            <dynamics damping="0.7"/>
+        </joint>
+        <transmission name="tran_r2">
+            <type>transmission_interface/SimpleTransmission</type>
+            <joint name="rh_r2">
+            <hardwareInterface>hardware_interface/EffortJointInterface</hardwareInterface>
+            </joint>
+            <actuator name="motor_r2">
+            <hardwareInterface>hardware_interface/EffortJointInterface</hardwareInterface>
+            <mechanicalReduction>1</mechanicalReduction>
+            </actuator>
+        </transmission>
+        <!-- rh_p12_rn_r2 -->
+        <link name="rh_p12_rn_r2">
+            <collision>
+            <origin xyz="0 0 0" rpy="0 0 0"/>
+            <geometry>
+                <mesh filename="file://$(find rh_p12_rn_description)/meshes/r2.stl" scale="0.001 0.001 0.001"/>
+            </geometry>
+            </collision>
+            <visual>
+            <origin xyz="0 0 0" rpy="0 0 0"/>
+            <geometry>
+                <mesh filename="file://$(find rh_p12_rn_description)/meshes/r2.stl" scale="0.001 0.001 0.001"/>
+            </geometry>
+            <material name="grey"/>
+            </visual>
+            <inertial>
+            <origin xyz="0.000 0.006 0.011" rpy="0 0 0"/>
+            <mass value="0.022"/>
+            <!--<inertia ixx="0.0" ixy="0.0" ixz="0.0" iyy="0.00001" iyz="0.0" izz="0.0" />-->
+            <inertia ixx="1.0" ixy="0.0" ixz="0.0" iyy="1.0" iyz="0.0" izz="1.0" />
+            </inertial>
+        </link>
+        <!-- Left Joint 1 -->
+        <joint name="rh_l1" type="revolute">
+            <parent link="rh_p12_rn_base"/>
+            <child link="rh_p12_rn_l1"/>
+            <origin xyz="0.0 -0.008 0.048" rpy="0 0 0"/>
+            <axis xyz="-1 0 0"/>
+            <limit velocity="6.5" effort="1000" lower="0.0" upper="1.1" />
+            <dynamics damping="0.7"/>
+        </joint>
+        <transmission name="tran_l1">
+            <type>transmission_interface/SimpleTransmission</type>
+            <joint name="rh_l1">
+            <hardwareInterface>hardware_interface/EffortJointInterface</hardwareInterface>
+            </joint>
+            <actuator name="motor_l1">
+            <hardwareInterface>hardware_interface/EffortJointInterface</hardwareInterface>
+            <mechanicalReduction>1</mechanicalReduction>
+            </actuator>
+        </transmission>
+        <!-- rh_p12_rn_l1 -->
+        <link name="rh_p12_rn_l1">
+            <collision>
+            <origin xyz="0 0 0" rpy="0 0 0"/>
+            <geometry>
+                <mesh filename="file://$(find rh_p12_rn_description)/meshes/l1.stl" scale="0.001 0.001 0.001"/>
+            </geometry>
+            </collision>
+            <visual>
+            <origin xyz="0 0 0" rpy="0 0 0"/>
+            <geometry>
+                <mesh filename="file://$(find rh_p12_rn_description)/meshes/l1.stl" scale="0.001 0.001 0.001"/>
+            </geometry>
+            <material name="grey"/>
+            </visual>
+            <inertial>
+            <origin xyz="0.000 -0.034 0.004" rpy="0 0 0"/>
+            <mass value="0.068"/>
+            <!--<inertia ixx="0.00004" ixy="0.0" ixz="0.0" iyy="0.00002" iyz="0.00001" izz="0.00002" />-->
+            <inertia ixx="1.0" ixy="0.0" ixz="0.0" iyy="1.0" iyz="0.0" izz="1.0" />
+            </inertial>
+        </link>
+        <!-- Left Joint 2 -->
+        <joint name="rh_l2" type="revolute">
+            <parent link="rh_p12_rn_l1"/>
+            <child link="rh_p12_rn_l2"/>
+            <origin xyz="0.0 -0.0493634 0.0285" rpy="0 0 0"/>
+            <axis xyz="1 0 0"/>
+            <limit velocity="6.5" effort="1000" lower="0.0" upper="1.0" />
+            <dynamics damping="0.7"/>
+        </joint>
+        <transmission name="tran_l2">
+            <type>transmission_interface/SimpleTransmission</type>
+            <joint name="rh_l2">
+            <hardwareInterface>hardware_interface/EffortJointInterface</hardwareInterface>
+            </joint>
+            <actuator name="motor_l2">
+            <hardwareInterface>hardware_interface/EffortJointInterface</hardwareInterface>
+            <mechanicalReduction>1</mechanicalReduction>
+            </actuator>
+        </transmission>
+        <!-- rh_p12_rn_l2 -->
+        <link name="rh_p12_rn_l2">
+            <collision>
+            <origin xyz="0 0 0" rpy="0 0 0"/>
+            <geometry>
+                <mesh filename="file://$(find rh_p12_rn_description)/meshes/l2.stl" scale="0.001 0.001 0.001"/>
+            </geometry>
+            </collision>
+            <visual>
+            <origin xyz="0 0 0" rpy="0 0 0"/>
+            <geometry>
+                <mesh filename="file://$(find rh_p12_rn_description)/meshes/l2.stl" scale="0.001 0.001 0.001"/>
+            </geometry>
+            <material name="grey"/>
+            </visual>
+            <inertial>
+            <origin xyz="0.000 -0.006 0.011" rpy="0 0 0"/>
+            <mass value="0.022"/>
+            <!--<inertia ixx="0.0" ixy="0.0" ixz="0.0" iyy="0.00001" iyz="0.0" izz="0.0" />-->
+            <inertia ixx="1.0" ixy="0.0" ixz="0.0" iyy="1.0" iyz="0.0" izz="1.0" />
+            </inertial>
+        </link>
     </xacro:macro>
 </robot>

Commit message: reverted gripper description to og

File: rh_p12_rn_description/urdf/rh_p12_rn_macro.xacro (robot description, xacro)
@@ -39,4 +39,14 @@
             <dynamics damping="0.7"/>
         </joint>
+        <transmission name="tran_r1">
+            <type>transmission_interface/SimpleTransmission</type>
+            <joint name="rh_p12_rn">
+            <hardwareInterface>hardware_interface/EffortJointInterface</hardwareInterface>
+            </joint>
+            <actuator name="motor_r1">
+            <hardwareInterface>hardware_interface/EffortJointInterface</hardwareInterface>
+            <mechanicalReduction>1</mechanicalReduction>
+            </actuator>
+        </transmission>
         <!-- rh_p12_rn_r1 -->
         <link name="rh_p12_rn_r1">
@@ -70,4 +80,14 @@
             <dynamics damping="0.7"/>
         </joint>
+        <transmission name="tran_r2">
+            <type>transmission_interface/SimpleTransmission</type>
+            <joint name="rh_r2">
+            <hardwareInterface>hardware_interface/EffortJointInterface</hardwareInterface>
+            </joint>
+            <actuator name="motor_r2">
+            <hardwareInterface>hardware_interface/EffortJointInterface</hardwareInterface>
+            <mechanicalReduction>1</mechanicalReduction>
+            </actuator>
+        </transmission>
         <!-- rh_p12_rn_r2 -->
         <link name="rh_p12_rn_r2">
@@ -101,4 +121,14 @@
             <dynamics damping="0.7"/>
         </joint>
+        <transmission name="tran_l1">
+            <type>transmission_interface/SimpleTransmission</type>
+            <joint name="rh_l1">
+            <hardwareInterface>hardware_interface/EffortJointInterface</hardwareInterface>
+            </joint>
+            <actuator name="motor_l1">
+            <hardwareInterface>hardware_interface/EffortJointInterface</hardwareInterface>
+            <mechanicalReduction>1</mechanicalReduction>
+            </actuator>
+        </transmission>
         <!-- rh_p12_rn_l1 -->
         <link name="rh_p12_rn_l1">
@@ -132,4 +162,14 @@
             <dynamics damping="0.7"/>
         </joint>
+        <transmission name="tran_l2">
+            <type>transmission_interface/SimpleTransmission</type>
+            <joint name="rh_l2">
+            <hardwareInterface>hardware_interface/EffortJointInterface</hardwareInterface>
+            </joint>
+            <actuator name="motor_l2">
+            <hardwareInterface>hardware_interface/EffortJointInterface</hardwareInterface>
+            <mechanicalReduction>1</mechanicalReduction>
+            </actuator>
+        </transmission>
         <!-- rh_p12_rn_l2 -->
         <link name="rh_p12_rn_l2">
