Commit message: robot bringup package update

File: robot_bringup/urdf/robot_arm_controlled.urdf.xacro (robot description, xacro)
@@ -1,8 +1,8 @@
 <?xml version="1.0"?>
 <robot name="my_robot_cell" xmlns:xacro="http://ros.org/wiki/xacro">
-  <!--First, include the macro from our custom description-->
-  <xacro:include filename="$(find my_robot_cell_description)/urdf/my_robot_cell_macro.xacro"/>
+  <xacro:include filename="$(find ur_description)/urdf/ur_macro.xacro"/>
   <!--The driver already provides a control tag for the UR arm, we can directly include-->
   <xacro:include filename="$(find ur_robot_driver)/urdf/ur.ros2_control.xacro"/>
+  <xacro:include filename="$(find rh_p12_rn_description)/urdf/rh_p12_rn_macro.xacro"/>
   <!--We need to specify the arguments used for parametrizing our description-->
   <xacro:arg name="ur_type" default="ur20"/>
@@ -19,7 +19,39 @@
   <xacro:arg name="mock_sensor_commands" default="false" />
   <link name="world" />
+  <joint type="fixed" name="workspace_joint">
+    <origin xyz="0 0 1.015" rpy="0 0 -1.5708"/>
+    <child link="workspace_link"/>
+    <parent link="world"/>
+  </joint>
+  <link name='workspace_link'>
+    <inertial>
+      <mass value="1.0e-03"/>
+      <origin xyz="0 0 0" rpy="0 0 0"/>
+      <inertia
+          ixx="1e-6" ixy="0" ixz="0"
+          iyy="1e-6" iyz="0"
+          izz="1e-6"
+      />
+    </inertial>
+  </link>
+  <joint type="fixed" name="camera_joint_optical">
+    <origin xyz="0 0 1" rpy="0 0 0"/>
+    <child link="camera_link_optical"/>
+    <parent link="workspace_link"/>
+  </joint>
+  <link name='camera_link_optical'>
+    <inertial>
+      <mass value="1.0e-03"/>
+      <origin xyz="0 0 0" rpy="0 0 0"/>
+      <inertia
+          ixx="1e-6" ixy="0" ixz="0"
+          iyy="1e-6" iyz="0"
+          izz="1e-6"
+      />
+    </inertial>
+  </link>
   <link name="robot_mount"/>
   <joint name="base_to_robot_mount" type="fixed">
-    <parent link="world"/>
+    <parent link="workspace_link"/>
     <child link="robot_mount"/>
     <origin xyz="0 0 0" rpy="0 0 ${pi}" />
@@ -37,4 +69,37 @@
     <origin xyz="0 0 0" rpy="0 0 0" />          <!-- position robot in the world -->
   </xacro:ur_robot>
+  <joint type="fixed" name="table_camera_joint">
+    <origin xyz="-1.1 -0.1 2.13" rpy="0 0.86 0"/>
+    <child link="table_camera_link"/>
+    <parent link="world"/>
+  </joint>
+  <link name='table_camera_link'>
+    <pose>0 0 0 0 0 0</pose>
+    <inertial>
+      <mass value="1.0e-03"/>
+      <origin xyz="0 0 0" rpy="0 0 0"/>
+      <inertia
+          ixx="1e-6" ixy="0" ixz="0"
+          iyy="1e-6" iyz="0"
+          izz="1e-6"
+      />
+    </inertial>
+    <visual>
+      <origin xyz="0 0 0" rpy="0 0 0"/>
+      <geometry>
+        <box size=".05 .05 .05"/>
+      </geometry>
+      <material name="red">
+        <color rgba="0.0 0.0 0.8 1.0"/>
+      </material>
+    </visual>
+  </link>
+  <joint type="fixed" name="table_camera_optical_joint">
+    <origin xyz="0 0 0" rpy="-1.5707 0 -1.5707"/>
+    <child link="table_camera_link_optical"/>
+    <parent link="table_camera_link"/>
+  </joint>
+  <link name="table_camera_link_optical">
+  </link>
   <!--Create the control tag for the UR robot-->
   <xacro:ur_ros2_control

Commit message: robot bringup package update

File: robot_bringup/urdf/robot_arm_controlled.urdf.xacro (robot description, xacro)
@@ -4,7 +4,9 @@
   <!--The driver already provides a control tag for the UR arm, we can directly include-->
   <xacro:include filename="$(find ur_robot_driver)/urdf/ur.ros2_control.xacro"/>
-  <xacro:include filename="$(find rh_p12_rn_description)/urdf/rh_p12_rn_macro.xacro"/>
+  <xacro:include filename="$(find rh_p12_rn_a_description)/urdf/rh_p12_rn_a.xacro" />
+  <xacro:include filename="$(find rh_p12_rn_a_description)/gazebo/rh_p12_rn_a.gazebo.xacro" />
+  <xacro:include filename="$(find rh_p12_rn_a_description)/ros2_control/rh_p12_rn_a.ros2_control.xacro" />
   <!--We need to specify the arguments used for parametrizing our description-->
-  <xacro:arg name="ur_type" default="ur20"/>
+  <xacro:arg name="ur_type" default="ur5e"/>
   <xacro:arg name="joint_limit_parameters_file" default="$(find ur_description)/config/$(arg ur_type)/joint_limits.yaml"/>
   <xacro:arg name="kinematics_parameters_file" default="$(find ur_description)/config/$(arg ur_type)/default_kinematics.yaml"/>
@@ -18,4 +20,6 @@
   <xacro:arg name="use_mock_hardware" default="false" />
   <xacro:arg name="mock_sensor_commands" default="false" />
+  <xacro:arg name="use_fake_hardware" default="false" />
+  <xacro:arg name="use_sim" default="false" />
   <link name="world" />
   <joint type="fixed" name="workspace_joint">
@@ -102,4 +106,10 @@
   <link name="table_camera_link_optical">
   </link>
+  <!--joint name="gripper_joint" type="fixed">
+    <parent link="$(arg ur_type)_tool0"/>
+    <child link="$(arg ur_type)_rh_p12_rn_base"/>
+    <origin xyz="0 0 0" rpy="0 0 0"/>
+  </joint-->
+  <!--xacro:rh_p12_rn_a prefix="$(arg ur_type)_" /-->
   <!--Create the control tag for the UR robot-->
   <xacro:ur_ros2_control
@@ -116,3 +126,7 @@
   />
   <!--If you had more controlled devices in your description, e.g. a gripper, you can add another ros2_control tag here-->
+  <!--xacro:rh_p12_rn_a_system
+    name="RH-P12-RN-A-System" prefix="$(arg ur_type)_" use_sim="$(arg use_sim)"
+    use_fake_hardware="$(arg use_fake_hardware)"
+    fake_sensor_commands="$(arg mock_sensor_commands)"/-->
 </robot>
