Commit message: rh_p12_rn_a custom decription package
moveit config

File: ur_moveit_config/config/ur.ros2_control.xacro (robot description, xacro)
@@ -50,29 +50,8 @@
                 <state_interface name="velocity"/>
             </joint>
-            <joint name="rh_l1">
+            <joint name="rh_r1">
                 <command_interface name="position"/>
                 <state_interface name="position">
-                  <param name="initial_value">${initial_positions['rh_l1']}</param>
-                </state_interface>
-                <state_interface name="velocity"/>
-            </joint>
-            <joint name="rh_l2">
-                <command_interface name="position"/>
-                <state_interface name="position">
-                  <param name="initial_value">${initial_positions['rh_l2']}</param>
-                </state_interface>
-                <state_interface name="velocity"/>
-            </joint>
-            <joint name="rh_p12_rn">
-                <command_interface name="position"/>
-                <state_interface name="position">
-                  <param name="initial_value">${initial_positions['rh_p12_rn']}</param>
-                </state_interface>
-                <state_interface name="velocity"/>
-            </joint>
-            <joint name="rh_r2">
-                <command_interface name="position"/>
-                <state_interface name="position">
-                  <param name="initial_value">${initial_positions['rh_r2']}</param>
+                  <param name="initial_value">${initial_positions['rh_r1']}</param>
                 </state_interface>
                 <state_interface name="velocity"/>

File: workspace_sim/urdf/robot_arm_moveit.urdf.xacro (robot description, xacro)
@@ -5,4 +5,6 @@
   <xacro:include filename="$(find ur_description)/urdf/inc/ur_joint_control.xacro" />
   <xacro:include filename="$(find rh_p12_rn_description)/urdf/joint_control.xacro" />
+  <xacro:include filename="$(find rh_p12_rn_a_description_custom)/urdf/rh_p12_rn_a.xacro" />
+  <xacro:include filename="$(find rh_p12_rn_a_description)/ros2_control/rh_p12_rn_a.ros2_control.xacro" />
   <xacro:arg name="ur_type" default="ur5e"/>
   <!-- parameters -->
@@ -18,4 +20,7 @@
   <xacro:arg name="simulation_controllers" default="" />
   <xacro:arg name="ros_namespace" default="" />
+  <xacro:arg name="use_sim" default="true" />
+  <xacro:arg name="use_fake_hardware" default="false" />
+  <xacro:arg name="fake_sensor_commands" default="false" />
   <link name="world"/>
   <joint type="fixed" name="workspace_joint">
@@ -41,13 +46,13 @@
     </inertial>
   </link>
-  <joint type="fixed" name="camera_joint">
+  <joint type="fixed" name="camera_joint_optical">
     <origin xyz="0 0 1" rpy="0 0 0"/>
-    <child link="camera_link"/>
+    <child link="camera_link_optical"/>
     <parent link="workspace_link"/>
   </joint>
-  <link name='camera_link'>
+  <link name='camera_link_optical'>
     <inertial>
       <mass value="1.0e-03"/>
-      <origin xyz="-0.6 0 1.63" rpy="0 0.86 0"/>
+      <origin xyz="0 0 0" rpy="0 0 0"/>
       <inertia
           ixx="1e-6" ixy="0" ixz="0"
@@ -79,5 +84,10 @@
     <origin xyz="0 0 0" rpy="0 0 0" />          <!-- position robot in the world -->
   </xacro:ur_robot>
-  <xacro:rh_p12_rn parent="$(arg tf_prefix)tool0"/>
+  <joint name="$(arg tf_prefix)gripper_joint" type="fixed">
+    <parent link="tool0"/>
+    <child link="$(arg tf_prefix)rh_p12_rn_base"/>
+    <origin xyz="0 0 0" rpy="0 0 0"/>
+  </joint>
+  <xacro:rh_p12_rn_a prefix="$(arg tf_prefix)" />
   <!-- End effector -->
   <joint name="end_effector_joint" type="fixed">
